Commit message: Update robot description

File: description/gazebo_friction.xacro (robot description, xacro)
@@ -1,61 +1,59 @@
 <?xml version="1.0"?>
 <robot xmlns:xacro="http://www.ros.org/wiki/xacro" xmlns:gz="http://gazebosim.org/schema">
-    <!-- Wheel friction macro -->
-    <gazebo reference='fl_wheel_link'>
-        <collision>
-          <surface>
-            <friction>
-              <ode>
-                <mu>1.5</mu>
-                <mu2>0.0</mu2>
-                <fdir1 gz:expressed_in="base_footprint">1 -1 0</fdir1>
-              </ode>
-            </friction>
-          </surface>
-        </collision>
-      </gazebo>
-      <gazebo reference='rl_wheel_link'>
-        <collision>
-          <surface>
-            <friction>
-              <ode>
-                <mu>1.5</mu>
-                <mu2>0.0</mu2>
-                <fdir1 gz:expressed_in="base_footprint">1 1 0</fdir1>
-              </ode>
-            </friction>
-          </surface>
-        </collision>
-      </gazebo>
-      <gazebo reference='fr_wheel_link'>
-        <collision>
-          <surface>
-            <friction>
-              <ode>
-                <mu>1.5</mu>
-                <mu2>0.0</mu2>
-                <fdir1 gz:expressed_in="base_footprint">1 1 0</fdir1>
-              </ode>
-            </friction>
-          </surface>
-        </collision>
-      </gazebo>
-      <gazebo reference='rr_wheel_link'>
-        <collision>
-          <surface>
-            <friction>
-              <ode>
-                <mu>1.5</mu>
-                <mu2>0.0</mu2>
-                <fdir1 gz:expressed_in="base_footprint">1 -1 0</fdir1>
-              </ode>
-            </friction>
-          </surface>
-        </collision>
-      </gazebo>
-      <gazebo reference="base_link">
-        <mu1>0.000002</mu1>
-        <mu2>0.000002</mu2>
-        <!-- <material>Gazebo/Red</material> -->
-      </gazebo>
+  <gazebo reference='fl_wheel_link'>
+    <collision>
+      <surface>
+        <friction>
+          <ode>
+            <mu>1.5</mu>
+            <mu2>0.0</mu2>
+            <fdir1 gz:expressed_in="base_footprint">1 -1 0</fdir1>
+          </ode>
+        </friction>
+      </surface>
+    </collision>
+  </gazebo>
+  <gazebo reference='rl_wheel_link'>
+    <collision>
+      <surface>
+        <friction>
+          <ode>
+            <mu>1.5</mu>
+            <mu2>0.0</mu2>
+            <fdir1 gz:expressed_in="base_footprint">1 1 0</fdir1>
+          </ode>
+        </friction>
+      </surface>
+    </collision>
+  </gazebo>
+  <gazebo reference='fr_wheel_link'>
+    <collision>
+      <surface>
+        <friction>
+          <ode>
+            <mu>1.5</mu>
+            <mu2>0.0</mu2>
+            <fdir1 gz:expressed_in="base_footprint">1 1 0</fdir1>
+          </ode>
+        </friction>
+      </surface>
+    </collision>
+  </gazebo>
+  <gazebo reference='rr_wheel_link'>
+    <collision>
+      <surface>
+        <friction>
+          <ode>
+            <mu>1.5</mu>
+            <mu2>0.0</mu2>
+            <fdir1 gz:expressed_in="base_footprint">1 -1 0</fdir1>
+          </ode>
+        </friction>
+      </surface>
+    </collision>
+  </gazebo>
+  <gazebo reference="base_link">
+    <mu1>0.000002</mu1>
+    <mu2>0.000002</mu2>
+  </gazebo>
 </robot>

File: description/lidar.xacro (robot description, xacro)
@@ -1,13 +1,36 @@
 <?xml version="1.0"?>
 <robot xmlns:xacro="http://www.ros.org/wiki/xacro">
+    <joint name="lidar_chassis_joint" type="fixed">
+        <parent link="chassis_link"/>
+        <child link="lidar_link"/>
+        <origin xyz="0.0 0 ${(chassis_z+lidar_z)/2 + chassis_visual_offset_z}" rpy="0 0 ${pi/2}"/>
+    </joint>
+    <link name="lidar_link">
+        <visual>
+            <origin xyz="0 0 0" rpy="0 0 0" />
+            <geometry>
+                <box size="${lidar_x} ${lidar_y} ${lidar_z}"/>
+            </geometry>
+            <material name="orange"/>
+        </visual>
+        <collision>
+            <origin xyz="0 0 0" rpy="0 0 0" />
+            <geometry>
+                <box size="${lidar_x} ${lidar_y} ${lidar_z}"/>
+            </geometry>
+        </collision>
+        <xacro:inertial_box mass="0.1" x="${lidar_x}" y="${lidar_y}" z="${lidar_z}">
+            <origin xyz="0.0 0.0 0.0" rpy="0.0 0.0 0.0"/>
+        </xacro:inertial_box>
+    </link>
     <joint name="lidar_joint" type="fixed">
-        <parent link="chassis_link"/>
+        <parent link="lidar_link"/>
         <child link="laser_frame"/>
-        <origin xyz="0.0 0 0.115" rpy="0 0 0"/>
+        <origin xyz="${lidar_x_offset} 0 ${(lidar_z+lidar_length)/2}" rpy="0 0 ${pi}"/>
     </joint>
     <link name="laser_frame">
         <visual>
             <geometry>
-                <cylinder radius="0.05" length="0.04"/>
+                <cylinder radius="${lidar_radius}" length="${lidar_length}"/>
             </geometry>
             <material name="red"/>
@@ -15,35 +38,37 @@
         <collision>
             <geometry>
-                <cylinder radius="0.05" length="0.04"/>
+                <cylinder radius="${lidar_radius}" length="${lidar_length}"/>
             </geometry>
         </collision>
-        <xacro:inertial_cylinder mass="0.1" length="0.04" radius="0.05">
+        <xacro:inertial_cylinder mass="0.05" length="${lidar_length}" radius="${lidar_radius}">
             <origin xyz="0 0 0" rpy="0 0 0"/>
         </xacro:inertial_cylinder>
     </link>
-    <gazebo reference="laser_frame">
-        <sensor name="laser" type="gpu_lidar">
-            <pose> 0 0 0 0 0 0 </pose>
-            <always_on>true</always_on>
-            <visualize>true</visualize>
-            <update_rate>10</update_rate>
-            <lidar>
-                <scan>
-                    <horizontal>
-                        <samples>360</samples>
-                        <resolution>1</resolution>
-                        <min_angle>-3.14159</min_angle>
-                        <max_angle>3.14159</max_angle>
-                    </horizontal>
-                </scan>
-                <range>
-                    <min>0.3</min>
-                    <max>12</max>
-                    <resolution>0.01</resolution>
-                </range>
-            </lidar>
-            <topic>scan</topic>
-            <gz_frame_id>laser_frame</gz_frame_id>
-        </sensor>
-    </gazebo>
+    <xacro:if value="$(arg use_sim)">
+        <gazebo reference="laser_frame">
+            <sensor name="laser" type="gpu_lidar">
+                <pose> 0 0 0 0 0 0 </pose>
+                <always_on>true</always_on>
+                <visualize>true</visualize>
+                <update_rate>10</update_rate>
+                <lidar>
+                    <scan>
+                        <horizontal>
+                            <samples>360</samples>
+                            <resolution>1</resolution>
+                            <min_angle>-${pi}</min_angle>
+                            <max_angle>${pi}</max_angle>
+                        </horizontal>
+                    </scan>
+                    <range>
+                        <min>0.3</min>
+                        <max>12</max>
+                        <resolution>0.01</resolution>
+                    </range>
+                </lidar>
+                <topic>scan</topic>
+                <gz_frame_id>laser_frame</gz_frame_id>
+            </sensor>
+        </gazebo>
+    </xacro:if>
 </robot>

File: description/properties.xacro (robot description, xacro)
@@ -1,16 +1,26 @@
 <?xml version="1.0"?>
 <robot xmlns:xacro="http://www.ros.org/wiki/xacro">
-    <xacro:property name="chassis_x" value="0.5"/>
-    <xacro:property name="chassis_y" value="0.4"/>
-    <xacro:property name="chassis_z" value="0.15"/>
-    <xacro:property name="chassis_visual_offset_z" value="0.02"/>
+    <xacro:property name="chassis_x" value="0.23"/>
+    <xacro:property name="chassis_y" value="0.15"/>
+    <xacro:property name="chassis_z" value="0.05"/>
+    <xacro:property name="chassis_visual_offset_z" value="0.005"/>
     <xacro:property name="chassis_mass" value="1.0"/>
-    <xacro:property name="base_link_offset_z" value="0.1"/>
-    <xacro:property name="wheel_radius" value="0.1"/>
-    <xacro:property name="wheel_length" value="0.1"/>
+    <xacro:property name="base_link_offset_z" value="0.04"/>
+    <xacro:property name="wheel_radius" value="0.04"/>
+    <xacro:property name="wheel_length" value="0.04"/>
     <xacro:property name="wheel_mass" value="0.2"/>
-    <xacro:property name="wheel_offset_x" value="0.15"/>
-    <xacro:property name="wheel_offset_y" value="0.25"/>
-    <xacro:property name="wheelbase" value="0.3"/>
-    <xacro:property name="wheellength" value="0.5"/>
+    <xacro:property name="wheel_stl_scale" value="0.0008 0.0008 0.0008"/>
+    <xacro:property name="wheelbase" value="0.174"/>
+    <xacro:property name="wheellength" value="0.204"/>
+    <xacro:property name="wheel_offset_x" value="${wheelbase/2}"/>
+    <xacro:property name="wheel_offset_y" value="${wheellength/2}"/>
+    <xacro:property name="effort" value="0.5" />
+    <xacro:property name="velocity" value="10.0" />
+    <xacro:property name="axle_radius" value="0.008"/>
+    <xacro:property name="lidar_x" value="0.11" />
+    <xacro:property name="lidar_y" value="0.07" />
+    <xacro:property name="lidar_z" value="0.07" />
+    <xacro:property name="lidar_x_offset" value="0.007" />
+    <xacro:property name="lidar_radius" value="0.035" />
+    <xacro:property name="lidar_length" value="0.025" />
 </robot>

File: description/robot.urdf.xacro (robot description, xacro)
@@ -1,12 +1,23 @@
 <?xml version="1.0"?>
 <robot xmlns:xacro="http://www.ros.org/wiki/xacro" name="robot">
+    <!-- args -->
     <xacro:arg name="use_ros2_control" default="true"/>
-    <xacro:include filename="robot_core.xacro"/>
+    <xacro:arg name="use_sim" default="false"/>
+    <!-- definitions -->
+    <xacro:include filename="$(find mecanum_robot)/description/properties.xacro"/>
+    <xacro:include filename="$(find mecanum_robot)/description/inertia_macros.xacro"/>
+    <xacro:include filename="$(find mecanum_robot)/description/materials.xacro"/>
+    <xacro:if value="$(arg use_sim)">
+        <xacro:include filename="$(find mecanum_robot)/description/gazebo_friction.xacro"/>
+    </xacro:if>
+    <!-- robot core and sensors -->
+    <xacro:include filename="$(find mecanum_robot)/description/robot_core.xacro"/>
+    <xacro:include filename="$(find mecanum_robot)/description/lidar.xacro"/>
+    <!-- controllers -->
     <xacro:if value="$(arg use_ros2_control)">
-        <xacro:include filename="ros2_control.xacro"/>
+        <xacro:include filename="$(find mecanum_robot)/description/ros2_control.xacro"/>
     </xacro:if>
     <xacro:unless value="$(arg use_ros2_control)">
-        <xacro:include filename="gazebo_control.xacro"/>
+        <xacro:include filename="$(find mecanum_robot)/description/gazebo_control.xacro"/>
     </xacro:unless>
-    <xacro:include filename="lidar.xacro"/>
 </robot>

File: description/robot_core.xacro (robot description, xacro)
@@ -1,11 +1,7 @@
 <?xml version="1.0"?>
 <robot xmlns:xacro="http://www.ros.org/wiki/xacro">
-  <xacro:include filename="properties.xacro"/>
-  <xacro:include filename="inertia_macros.xacro"/>
-  <xacro:include filename="materials.xacro"/>
-  <xacro:include filename="gazebo_friction.xacro"/>
     <!-- base and base footprint -->
     <link name="base_footprint"/>
-    <joint name="base_footprint_oint" type="fixed">
+    <joint name="base_footprint_joint" type="fixed">
       <origin xyz="0.0 0.0 ${base_link_offset_z}" rpy="0.0 0.0 0.0"/>
       <parent link="base_footprint"/>
@@ -37,4 +33,76 @@
       </collision>
     </link>
+    <!-- Front left axle -->
+    <joint name="fl_axle_joint" type="fixed">
+      <origin xyz="${wheel_offset_x} ${(chassis_y/2 + wheel_offset_y)/2} 0.0" rpy="0.0 0.0 0.0"/>
+      <parent link="base_link"/>
+      <child link="fl_axle_link"/>
+    </joint>
+    <link name="fl_axle_link">
+      <xacro:inertial_cylinder mass="0.01" length="${wheel_offset_y - chassis_y/2}" radius="${axle_radius}">
+        <origin xyz="0.0 0.0 0.0" rpy="0.0 0.0 0.0"/>
+      </xacro:inertial_cylinder>
+      <visual>
+        <origin xyz="0.0 0.0 0.0" rpy="${pi/2} 0.0 0.0"/>
+        <geometry>
+          <cylinder radius="${axle_radius}" length="${wheel_offset_y - chassis_y/2}"/>
+        </geometry>
+        <material name="black"/>
+      </visual>
+    </link>
+    <!-- Rear left axle -->
+    <joint name="rl_axle_joint" type="fixed">
+      <origin xyz="-${wheel_offset_x} ${(chassis_y/2 + wheel_offset_y)/2} 0.0" rpy="0.0 0.0 0.0"/>
+      <parent link="base_link"/>
+      <child link="rl_axle_link"/>
+    </joint>
+    <link name="rl_axle_link">
+      <xacro:inertial_cylinder mass="0.01" length="${wheel_offset_y - chassis_y/2}" radius="${axle_radius}">
+        <origin xyz="0.0 0.0 0.0" rpy="0.0 0.0 0.0"/>
+      </xacro:inertial_cylinder>
+      <visual>
+        <origin xyz="0.0 0.0 0.0" rpy="${pi/2} 0.0 0.0"/>
+        <geometry>
+          <cylinder radius="${axle_radius}" length="${wheel_offset_y - chassis_y/2}"/>
+        </geometry>
+        <material name="black"/>
+      </visual>
+    </link>
+    <!-- Front right axle -->
+    <joint name="fr_axle_joint" type="fixed">
+      <origin xyz="${wheel_offset_x} -${(chassis_y/2 + wheel_offset_y)/2} 0.0" rpy="0.0 0.0 0.0"/>
+      <parent link="base_link"/>
+      <child link="fr_axle_link"/>
+    </joint>
+    <link name="fr_axle_link">
+      <xacro:inertial_cylinder mass="0.01" length="${wheel_offset_y - chassis_y/2}" radius="${axle_radius}">
+        <origin xyz="0.0 0.0 0.0" rpy="0.0 0.0 0.0"/>
+      </xacro:inertial_cylinder>
+      <visual>
+        <origin xyz="0.0 0.0 0.0" rpy="${pi/2} 0.0 0.0"/>
+        <geometry>
+          <cylinder radius="${axle_radius}" length="${wheel_offset_y - chassis_y/2}"/>
+        </geometry>
+        <material name="black"/>
+      </visual>
+    </link>
+    <!-- Rear right axle -->
+    <joint name="rr_axle_joint" type="fixed">
+      <origin xyz="-${wheel_offset_x} -${(chassis_y/2 + wheel_offset_y)/2} 0.0" rpy="0.0 0.0 0.0"/>
+      <parent link="base_link"/>
+      <child link="rr_axle_link"/>
+    </joint>
+    <link name="rr_axle_link">
+      <xacro:inertial_cylinder mass="0.01" length="${wheel_offset_y - chassis_y/2}" radius="${axle_radius}">
+        <origin xyz="0.0 0.0 0.0" rpy="0.0 0.0 0.0"/>
+      </xacro:inertial_cylinder>
+      <visual>
+        <origin xyz="0.0 0.0 0.0" rpy="${pi/2} 0.0 0.0"/>
+        <geometry>
+          <cylinder radius="${axle_radius}" length="${wheel_offset_y - chassis_y/2}"/>
+        </geometry>
+        <material name="black"/>
+      </visual>
+    </link>
     <!-- Front left wheel-->
     <joint name="fl_wheel_joint" type="continuous">
@@ -43,5 +111,5 @@
       <child link="fl_wheel_link"/>
       <axis xyz="0.0 0.0 1"/>
-      <limit effort="0.5" velocity="10.0"/>
+      <limit effort="${effort}" velocity="${velocity}"/>
     </joint>
     <link name="fl_wheel_link">
@@ -49,9 +117,9 @@
         <origin xyz="0.0 0.0 0.0" rpy="0.0 0.0 0.0"/>
       </xacro:inertial_cylinder>
-      <visual name="">
-        <origin xyz="0.0 0.0 0.0" rpy="${pi/2} 0.0 0.0"/>
-        <geometry>
-          <!-- <sphere radius=".1"/> -->
-          <mesh filename="package://mecanum_robot/meshes/mecanum_wheel_left.STL" scale="0.002 .002 0.002"/>
+      <visual>
+        <origin xyz="0.0 0.0 0.0" rpy="${pi/2} 0.0 0.0"/>
+        <geometry>
+          <!-- <sphere radius=".04"/> -->
+          <mesh filename="package://mecanum_robot/meshes/mecanum_wheel_left.STL" scale="${wheel_stl_scale}"/>
         </geometry>
         <material name="blue"/>
@@ -69,5 +137,5 @@
       <child link="rl_wheel_link"/>
       <axis xyz="0.0 0.0 1"/>
-      <limit effort="0.5" velocity="10.0"/>
+      <limit effort="${effort}" velocity="${velocity}"/>
     </joint>
     <link name="rl_wheel_link">
@@ -75,9 +143,9 @@
         <origin xyz="0.0 0.0 0.0" rpy="0.0 0.0 0.0"/>
       </xacro:inertial_cylinder>
-      <visual name="">
-        <origin xyz="0.0 0.0 0.0" rpy="${pi/2} 0.0 0.0"/>
-        <geometry>
-          <!-- <sphere radius=".1"/> -->
-          <mesh filename="package://mecanum_robot/meshes/mecanum_wheel_right.STL" scale="0.002 .002 0.002"/>
+      <visual>
+        <origin xyz="0.0 0.0 0.0" rpy="${pi/2} 0.0 0.0"/>
+        <geometry>
+          <!-- <sphere radius=".04"/> -->
+          <mesh filename="package://mecanum_robot/meshes/mecanum_wheel_right.STL" scale="${wheel_stl_scale}"/>
         </geometry>
         <material name="blue"/>
@@ -95,5 +163,5 @@
       <child link="fr_wheel_link"/>
       <axis xyz="0.0 0.0 -1"/>
-      <limit effort="0.5" velocity="10.0"/>
+      <limit effort="${effort}" velocity="${velocity}"/>
     </joint>
     <link name="fr_wheel_link">
@@ -101,9 +169,9 @@
         <origin xyz="0.0 0.0 0.0" rpy="0.0 0.0 0.0"/>
       </xacro:inertial_cylinder>
-      <visual name="">
-        <origin xyz="0.0 0.0 0.0" rpy="${pi/2} 0.0 0.0"/>
-        <geometry>
-          <!-- <sphere radius=".1"/> -->
-          <mesh filename="package://mecanum_robot/meshes/mecanum_wheel_right.STL" scale="0.002 .002 0.002"/>
+      <visual>
+        <origin xyz="0.0 0.0 0.0" rpy="${pi/2} 0.0 0.0"/>
+        <geometry>
+          <!-- <sphere radius=".04"/> -->
+          <mesh filename="package://mecanum_robot/meshes/mecanum_wheel_right.STL" scale="${wheel_stl_scale}"/>
         </geometry>
         <material name="blue"/>
@@ -121,5 +189,5 @@
       <child link="rr_wheel_link"/>
       <axis xyz="0.0 0.0 -1"/>
-      <limit effort="0.5" velocity="10.0"/>
+      <limit effort="${effort}" velocity="${velocity}"/>
     </joint>
     <link name="rr_wheel_link">
@@ -127,9 +195,9 @@
         <origin xyz="0.0 0.0 0.0" rpy="0.0 0.0 0.0"/>
       </xacro:inertial_cylinder>
-      <visual name="">
-        <origin xyz="0.0 0.0 0.0" rpy="${pi/2} 0.0 0.0"/>
-        <geometry>
-          <!-- <sphere radius=".1"/> -->
-          <mesh filename="package://mecanum_robot/meshes/mecanum_wheel_left.STL" scale="0.002 .002 0.002"/>
+      <visual>
+        <origin xyz="0.0 0.0 0.0" rpy="${pi/2} 0.0 0.0"/>
+        <geometry>
+          <!-- <sphere radius=".04"/> -->
+          <mesh filename="package://mecanum_robot/meshes/mecanum_wheel_left.STL" scale="${wheel_stl_scale}"/>
         </geometry>
         <material name="blue"/>

File: description/ros2_control.xacro (robot description, xacro)
@@ -1,5 +1,4 @@
 <?xml version="1.0"?>
 <robot xmlns:xacro="http://www.ros.org/wiki/xacro">
-    <xacro:arg name="use_sim" default="false"/>
     <ros2_control name="Mecanum_robot" type="system">
         <hardware>
@@ -13,7 +12,7 @@
                 <param name="rear_left_wheel_name">rl_wheel_joint</param>
                 <param name="rear_right_wheel_name">rr_wheel_joint</param>
-                <param name="device">/dev/ttyACM0</param>
+                <param name="device">/dev/ttyAMA0</param>
                 <param name="baud_rate">115200</param>
-                <param name="timeout_ms">1000</param>
+                <param name="timeout_ms">50</param>
                 <param name="kp">3.0</param>
                 <param name="ki">0.5</param>
@@ -23,6 +22,6 @@
         <joint name="fl_wheel_joint">
             <command_interface name="velocity">
-                <param name="min">-10</param>
-                <param name="max">10</param>
+                <param name="min">-${velocity}</param>
+                <param name="max">${velocity}</param>
             </command_interface>
             <state_interface name="position"/>
@@ -31,6 +30,6 @@
         <joint name="fr_wheel_joint">
             <command_interface name="velocity">
-                <param name="min">-10</param>
-                <param name="max">10</param>
+                <param name="min">-${velocity}</param>
+                <param name="max">${velocity}</param>
             </command_interface>
             <state_interface name="position"/>
@@ -39,6 +38,6 @@
         <joint name="rl_wheel_joint">
             <command_interface name="velocity">
-                <param name="min">-10</param>
-                <param name="max">10</param>
+                <param name="min">-${velocity}</param>
+                <param name="max">${velocity}</param>
             </command_interface>
             <state_interface name="position"/>
@@ -47,6 +46,6 @@
         <joint name="rr_wheel_joint">
             <command_interface name="velocity">
-                <param name="min">-10</param>
-                <param name="max">10</param>
+                <param name="min">-${velocity}</param>
+                <param name="max">${velocity}</param>
             </command_interface>
             <state_interface name="position"/>
