Commit message: Add gazebo plugins to control robot

File: description/properties.xacro (robot description, xacro)
@@ -12,5 +12,5 @@
     <xacro:property name="wheel_offset_x" value="0.15"/>
     <xacro:property name="wheel_offset_y" value="0.25"/>
-    <xacro:property name="wheelbase" value="0.1"/>
-    <xacro:property name="wheellength" value="0.1"/>
+    <xacro:property name="wheelbase" value="0.3"/>
+    <xacro:property name="wheellength" value="0.5"/>
 </robot>

File: description/robot.urdf.xacro (robot description, xacro)
@@ -2,3 +2,4 @@
 <robot xmlns:xacro="http://www.ros.org/wiki/xacro" name="robot">
     <xacro:include filename="robot_core.xacro"/>
+    <xacro:include filename="gazebo_control.xacro"/>
 </robot>

File: description/robot_core.xacro (robot description, xacro)
@@ -4,4 +4,5 @@
   <xacro:include filename="inertia_macros.xacro"/>
   <xacro:include filename="materials.xacro"/>
+  <xacro:include filename="gazebo_friction.xacro"/>
     <!-- base and base footprint -->
     <link name="base_footprint"/>
@@ -27,5 +28,5 @@
           <box size="${chassis_x} ${chassis_y} ${chassis_z}"/>
         </geometry>
-        <material name="red"/>
+        <material name="orange"/>
       </visual>
       <collision>

Commit message: Add ToF distance sensor integration with range sensor broadcaster

File: description/properties.xacro (robot description, xacro)
@@ -24,3 +24,6 @@
     <xacro:property name="lidar_radius" value="0.035" />
     <xacro:property name="lidar_length" value="0.025" />
+    <xacro:property name="tof_x" value="0.01" />
+    <xacro:property name="tof_y" value="0.02" />
+    <xacro:property name="tof_z" value="0.015" />
 </robot>

File: description/robot.urdf.xacro (robot description, xacro)
@@ -14,4 +14,5 @@
     <xacro:include filename="$(find mecanum_robot)/description/robot_core.xacro"/>
     <xacro:include filename="$(find mecanum_robot)/description/lidar.xacro"/>
+    <xacro:include filename="$(find mecanum_robot)/description/distance_sensor.xacro"/>
     <!-- controllers -->
     <xacro:if value="$(arg use_ros2_control)">

File: description/ros2_control.xacro (robot description, xacro)
@@ -22,4 +22,7 @@
         <sensor name="battery_state">
             <state_interface name="voltage" />
+        </sensor>
+        <sensor name="range_sensor">
+            <state_interface name="range" />
         </sensor>
         <joint name="fl_wheel_joint">
