Commit message: Fix lidar orientation and update dimensions; add second range sensor field

File: description/lidar.xacro (robot description, xacro)
@@ -4,5 +4,5 @@
         <parent link="chassis_link"/>
         <child link="lidar_link"/>
-        <origin xyz="0.0 0 ${(chassis_z+lidar_z)/2 + chassis_visual_offset_z}" rpy="0 0 ${pi/2}"/>
+        <origin xyz="${lidar_x_offset} 0 ${(chassis_z+lidar_z)/2 + chassis_visual_offset_z}" rpy="0 0 ${pi}"/>
     </joint>
     <link name="lidar_link">
@@ -27,5 +27,5 @@
         <parent link="lidar_link"/>
         <child link="laser_frame"/>
-        <origin xyz="${lidar_x_offset} 0 ${(lidar_z+lidar_length)/2}" rpy="0 0 ${pi}"/>
+        <origin xyz="${lidar_x_offset} 0 ${(lidar_z+lidar_length)/2}" rpy="0 0 0"/>
     </joint>
     <link name="laser_frame">

File: description/properties.xacro (robot description, xacro)
@@ -18,8 +18,8 @@
     <xacro:property name="velocity" value="10.0" />
     <xacro:property name="axle_radius" value="0.008"/>
-    <xacro:property name="lidar_x" value="0.11" />
-    <xacro:property name="lidar_y" value="0.07" />
-    <xacro:property name="lidar_z" value="0.07" />
-    <xacro:property name="lidar_x_offset" value="0.007" />
+    <xacro:property name="lidar_x" value="0.097" />
+    <xacro:property name="lidar_y" value="0.072" />
+    <xacro:property name="lidar_z" value="0.035" />
+    <xacro:property name="lidar_x_offset" value="0.012" />
     <xacro:property name="lidar_radius" value="0.035" />
     <xacro:property name="lidar_length" value="0.025" />

Commit message: Rotate lidar frame 180° to correct scan orientation

File: description/lidar.xacro (robot description, xacro)
@@ -27,5 +27,5 @@
         <parent link="lidar_link"/>
         <child link="laser_frame"/>
-        <origin xyz="${lidar_x_offset} 0 ${(lidar_z+lidar_length)/2}" rpy="0 0 0"/>
+        <origin xyz="${lidar_x_offset} 0 ${(lidar_z+lidar_length)/2}" rpy="0 0 ${pi}"/>
     </joint>
     <link name="laser_frame">
