Commit message: Add second ToF range sensor with dual broadcaster support

File: description/distance_sensor.xacro (robot description, xacro)
@@ -1,10 +1,33 @@
 <?xml version="1.0"?>
 <robot xmlns:xacro="http://www.ros.org/wiki/xacro">
-    <joint name="tof_joint" type="fixed">
+    <joint name="tof1_joint" type="fixed">
         <parent link="chassis_link"/>
-        <child link="tof_frame"/>
-        <origin xyz="${chassis_x/2 + tof_x/2} 0 ${chassis_visual_offset_z}" rpy="0 0 0"/>
+        <child link="tof1_frame"/>
+        <origin xyz="${chassis_x/2 + tof_x/2} ${tof_y_offset} ${chassis_visual_offset_z}" rpy="0 0 0"/>
     </joint>
-    <link name="tof_frame">
+    <link name="tof1_frame">
+        <visual>
+            <origin xyz="0 0 0" rpy="0 0 0"/>
+            <geometry>
+                <box size="${tof_x} ${tof_y} ${tof_z}"/>
+            </geometry>
+            <material name="red"/>
+        </visual>
+        <collision>
+            <origin xyz="0 0 0" rpy="0 0 0"/>
+            <geometry>
+                <box size="${tof_x} ${tof_y} ${tof_z}"/>
+            </geometry>
+        </collision>
+        <xacro:inertial_box mass="0.005" x="${tof_x}" y="${tof_y}" z="${tof_z}">
+            <origin xyz="0 0 0" rpy="0 0 0"/>
+        </xacro:inertial_box>
+    </link>
+    <joint name="tof2_joint" type="fixed">
+        <parent link="chassis_link"/>
+        <child link="tof2_frame"/>
+        <origin xyz="${chassis_x/2 + tof_x/2} -${tof_y_offset} ${chassis_visual_offset_z}" rpy="0 0 0"/>
+    </joint>
+    <link name="tof2_frame">
         <visual>
             <origin xyz="0 0 0" rpy="0 0 0"/>

File: description/properties.xacro (robot description, xacro)
@@ -27,3 +27,4 @@
     <xacro:property name="tof_y" value="0.02" />
     <xacro:property name="tof_z" value="0.015" />
+    <xacro:property name="tof_y_offset" value="0.02" />
 </robot>

File: description/ros2_control.xacro (robot description, xacro)
@@ -23,5 +23,8 @@
             <state_interface name="voltage" />
         </sensor>
-        <sensor name="range_sensor">
+        <sensor name="range_sensor_1">
+            <state_interface name="range" />
+        </sensor>
+        <sensor name="range_sensor_2">
             <state_interface name="range" />
         </sensor>

Commit message: Adjust ToF sensor placement with configurable offsets and rotation

File: description/distance_sensor.xacro (robot description, xacro)
@@ -4,5 +4,5 @@
         <parent link="chassis_link"/>
         <child link="tof1_frame"/>
-        <origin xyz="${chassis_x/2 + tof_x/2} ${tof_y_offset} ${chassis_visual_offset_z}" rpy="0 0 0"/>
+        <origin xyz="${chassis_x/2 + tof_x/2 + tof_x_offset} ${tof_y_offset} ${chassis_visual_offset_z + tof_z_offset}" rpy="0 0 ${tof_y_rot}"/>
     </joint>
     <link name="tof1_frame">
@@ -27,5 +27,5 @@
         <parent link="chassis_link"/>
         <child link="tof2_frame"/>
-        <origin xyz="${chassis_x/2 + tof_x/2} -${tof_y_offset} ${chassis_visual_offset_z}" rpy="0 0 0"/>
+        <origin xyz="${chassis_x/2 + tof_x/2 + tof_x_offset} -${tof_y_offset} ${chassis_visual_offset_z + tof_z_offset}" rpy="0 0 -${tof_y_rot}"/>
     </joint>
     <link name="tof2_frame">

File: description/properties.xacro (robot description, xacro)
@@ -27,4 +27,7 @@
     <xacro:property name="tof_y" value="0.02" />
     <xacro:property name="tof_z" value="0.015" />
+    <xacro:property name="tof_x_offset" value="-0.005" />
     <xacro:property name="tof_y_offset" value="0.02" />
+    <xacro:property name="tof_z_offset" value="-0.005" />
+    <xacro:property name="tof_y_rot" value="0.17453" />
 </robot>
